Commit message: Updating Jiqi URDF

File: src/articubot/jiqi_desc/jiqi_bot.urdf.xacro (robot description, xacro)
@@ -2,3 +2,4 @@
 <robot xmlns:xacro="http://www.ros.org/wiki/xacro" name="jiqi_bot">
     <xacro:include filename="jiqi_core.xacro"/>
+    <xacro:include filename="rplidar.xacro"/>
 </robot>

File: src/articubot/jiqi_desc/jiqi_core.xacro (robot description, xacro)
@@ -29,7 +29,5 @@
                 <box size="0.7 0.415 0.07"/>
             </geometry>
-            <material name="green">
-                <color rgba="0.2 1.0 0.2 1.0"/>
-            </material>
+            <material name="green"/>
         </visual>
         <collision>
@@ -58,4 +56,5 @@
                 <cylinder radius="0.09" length="0.05"/>
             </geometry>
+            <material name="black"/>
         </visual>
         <collision>
@@ -81,4 +80,5 @@
                 <cylinder radius="0.09" length="0.05"/>
             </geometry>
+            <material name="black"/>
         </visual>
         <collision>
@@ -104,4 +104,5 @@
                 <cylinder radius="0.09" length="0.05"/>
             </geometry>
+            <material name="black"/>
         </visual>
         <collision>
@@ -127,4 +128,5 @@
                 <cylinder radius="0.09" length="0.05"/>
             </geometry>
+            <material name="black"/>
         </visual>
         <collision>
@@ -138,8 +140,24 @@
     </link>
     <!-- Lidar Mount -->
-    <joint name="lidar_mount_joint">
-        <origin xyz="0.0 0.0 0.0" rpy="0.0 0.0 0.0"/>
+    <joint name="lidar_mount_joint" type="fixed">
+        <origin xyz="0.0 0.0 0.035" rpy="0.0 0.0 0.0"/>
         <parent link="chassis_link"/>
         <child link="lidar_mount_link"/>
     </joint>
+    <link name="lidar_mount_link">
+        <visual>
+            <origin xyz="0.0 0.0 0.04" rpy="0.0 0.0 0.0"/>
+            <geometry>
+                <box size="0.1 0.1 0.08"/>
+            </geometry>
+        </visual>
+        <collision>
+            <geometry>
+                <box size="0.1 0.1 0.08"/>
+            </geometry>
+        </collision>
+        <xacro:inertial_box mass="0.5" x="0.1" y="0.1" z="0.08">
+            <origin xyz="0.0 0.0 0.0" rpy="0.0 0.0 0.0"/>
+        </xacro:inertial_box>
+    </link>
 </robot>
