Commit message: Fixing Lidar Slam Path Planning

File: src/articubot/jiqi_desc/jiqi_core.xacro (robot description, xacro)
@@ -19,5 +19,5 @@
     <link name="base_link"></link>
     <joint name="base_joint" type="fixed">
-        <origin xyz="1.0 1.0 0.0" rpy="0.0 0.0 0.0"/>
+        <origin xyz="0.0 0.0 0.0" rpy="0.0 0.0 0.0"/>
         <parent link="base_link"/>
         <child link="chassis_link"/>
@@ -44,5 +44,5 @@
     </link>
     <!-- FRONT RIGHT WHEEL -->
-    <joint name="fr_wheel_joint" type="continuous">
+    <!-- <joint name="fr_wheel_joint" type="continuous">
         <parent link="chassis_link"/>
         <child link="fr_wheel_link"/>
@@ -66,7 +66,7 @@
             <origin xyz="0.0 0.0 0.0" rpy="0.0 0.0 0.0"/>
         </xacro:inertial_cylinder>
-    </link>
+    </link> -->
     <!-- FRONT LEFT WHEEL -->
-    <joint name="fl_wheel_joint" type="continuous">
+    <!-- <joint name="fl_wheel_joint" type="continuous">
         <parent link="chassis_link"/>
         <child link="fl_wheel_link"/>
@@ -90,7 +90,7 @@
             <origin xyz="0.0 0.0 0.0" rpy="0.0 0.0 0.0"/>
         </xacro:inertial_cylinder>
-    </link>
+    </link> -->
     <!-- BACK RIGHT WHEEL -->
-    <joint name="br_wheel_joint" type="continuous">
+    <!-- <joint name="br_wheel_joint" type="continuous">
         <parent link="chassis_link"/>
         <child link="br_wheel_link"/>
@@ -114,11 +114,12 @@
             <origin xyz="0.0 0.0 0.0" rpy="0.0 0.0 0.0"/>
         </xacro:inertial_cylinder>
-    </link>
+    </link> -->
     <!-- BACK LEFT WHEEL -->
+<!--
     <joint name="bl_wheel_joint" type="continuous">
         <parent link="chassis_link"/>
         <child link="bl_wheel_link"/>
         <axis xyz="0.0 0.0 -1.0"/>
-        <origin xyz="-0.29 -0.2325 0.025" rpy="${pi/2} 0.0 0.0"/>
+        <origin xyz="-0.29 -0.2325 0.025" rpy="<node pkg="rviz" type="rviz" name="rviz" args="-d $(find articubot)/rviz/hector_config.rviz"/> 0.0 0.0"/>
     </joint>
     <link name="bl_wheel_link">
@@ -138,8 +139,8 @@
             <origin xyz="0.0 0.0 0.0" rpy="0.0 0.0 0.0"/>
         </xacro:inertial_cylinder>
-    </link>
+    </link> -->
     <!-- Lidar Mount -->
     <joint name="lidar_mount_joint" type="fixed">
-        <origin xyz="0.0 0.0 0.035" rpy="0.0 0.0 0.0"/>
+        <origin xyz="0.3 0.0 0.035" rpy="0.0 0.0 0.0"/>
         <parent link="chassis_link"/>
         <child link="lidar_mount_link"/>

File: src/articubot/jiqi_desc/rplidar.xacro (robot description, xacro)
@@ -5,5 +5,5 @@
         <parent link="lidar_mount_link"/>
         <child link="laser"/>
-        <origin xyz="0.0 0.0 0.08" rpy="0.0 0.0 0.0"/>
+        <origin xyz="0.0 0.0 0.08" rpy="0.0 0.0 ${pi}"/>
     </joint>
     <link name="laser">
