Commit message: Teb Local Planner

File: src/articubot/description/lidar.xacro (robot description, xacro)
@@ -3,8 +3,8 @@
     <joint name="laser_joint" type="fixed">
         <parent link="chassis"/>
-        <child link="laser_frame"/>
+        <child link="laser"/>
         <origin xyz="0.1 0 0.175" rpy="0.0 0.0 0.0"/>
     </joint>
-    <link name="laser_frame">
+    <link name="laser">
         <visual>
             <geometry>
@@ -22,5 +22,5 @@
         </xacro:inertial_cylinder>
     </link>
-    <gazebo reference="laser_frame">
+    <gazebo reference="laser">
         <material>Gazebo/Red</material>
         <sensor name="laser" type="ray">
@@ -47,5 +47,5 @@
             <plugin name="laser_controller" filename="libgazebo_ros_laser.so">
                 <topicName>/scan</topicName>
-                <frameName>laser_frame</frameName>
+                <frameName>laser</frameName>
             </plugin>
         </sensor>
