Commit message: Jiqi URDF ZED_CAM update

File: src/articubot/description/gazebo_control.xacro (robot description, xacro)
@@ -5,5 +5,5 @@
             <!-- plugin config-->
             <robotBaseFrame>base_link</robotBaseFrame>
-            <updateRate>20</updateRate>
+            <updateRate>10.0</updateRate>
             <!-- wheel info-->
             <leftJoint>left_wheel_joint</leftJoint>
@@ -15,9 +15,10 @@
             <maxWheelAcceleration>10</maxWheelAcceleration>
             <!-- Output -->
-            <odometryFrame>odom123</odometryFrame> <!-- CHANGE BACK TO ODOM-->
-            <publishOdomTF>false</publishOdomTF> <!-- CHANGE BACK TO true-->
+            <odometryFrame>odom</odometryFrame> <!-- CHANGE BACK TO ODOM-->
+            <publishOdom>true</publishOdom> <!-- CHANGE BACK TO true-->
             <publishWheelTF>false</publishWheelTF> <!-- CHANGE BACK TO true-->
-            <odometryTopic>odom123</odometryTopic>
-            <publishTF>0</publishTF>
+            <odometryTopic>odom</odometryTopic>
+            <publishTF>1</publishTF>
+            <odometrySource>1</odometrySource>
         </plugin>
     </gazebo>

File: src/articubot/description/lidar.xacro (robot description, xacro)
@@ -25,5 +25,5 @@
         <material>Gazebo/Red</material>
         <sensor name="laser" type="ray">
-            <updateRate>20</updateRate>
+            <updateRate>10.0</updateRate>
             <visualize>false</visualize> <!-- to see lidar line in gazebo set to true-->
             <pose>0 0 0 0 0 0</pose>
@@ -40,5 +40,5 @@
                 </scan>
                 <range>
-                    <min>0.3</min>
+                    <min>0.1</min>
                     <max>12</max>
                     <resolution>0.01</resolution>

File: src/articubot/description/robot.urdf.xacro (robot description, xacro)
@@ -5,4 +5,4 @@
     <xacro:include filename="gazebo_control.xacro"/>
     <xacro:include filename="lidar.xacro"/>
-    <xacro:include filename="camera.xacro"/>
+    <!-- <xacro:include filename="camera.xacro"/> -->
 </robot>

File: src/articubot/jiqi_desc/jiqi_bot.urdf.xacro (robot description, xacro)
@@ -3,3 +3,4 @@
     <xacro:include filename="jiqi_core.xacro"/>
     <xacro:include filename="rplidar.xacro"/>
+    <xacro:include filename="zed_cam.xacro"/>
 </robot>

File: src/articubot/jiqi_desc/jiqi_core.xacro (robot description, xacro)
@@ -142,5 +142,5 @@
     <!-- Lidar Mount -->
     <joint name="lidar_mount_joint" type="fixed">
-        <origin xyz="0.3 0.0 0.035" rpy="0.0 0.0 0.0"/>
+        <origin xyz="0.225 0.0 0.035" rpy="0.0 0.0 0.0"/>
         <parent link="chassis_link"/>
         <child link="lidar_mount_link"/>
@@ -148,15 +148,15 @@
     <link name="lidar_mount_link">
         <visual>
-            <origin xyz="0.0 0.0 0.04" rpy="0.0 0.0 0.0"/>
+            <origin xyz="0.0 0.0 0.16" rpy="0.0 0.0 0.0"/>
             <geometry>
-                <box size="0.1 0.1 0.08"/>
+                <box size="0.25 0.3 0.25"/>
             </geometry>
         </visual>
         <collision>
             <geometry>
-                <box size="0.1 0.1 0.08"/>
+                <box size="0.25 0.3 0.25"/>
             </geometry>
         </collision>
-        <xacro:inertial_box mass="0.5" x="0.1" y="0.1" z="0.08">
+        <xacro:inertial_box mass="0.5" x="0.25" y="0.3" z="0.25">
             <origin xyz="0.0 0.0 0.0" rpy="0.0 0.0 0.0"/>
         </xacro:inertial_box>

File: src/articubot/jiqi_desc/rplidar.xacro (robot description, xacro)
@@ -5,5 +5,5 @@
         <parent link="lidar_mount_link"/>
         <child link="laser"/>
-        <origin xyz="0.0 0.0 0.08" rpy="0.0 0.0 ${pi}"/>
+        <origin xyz="0.07 0.0 0.29" rpy="0.0 0.0 ${pi}"/>
     </joint>
     <link name="laser">
